File: VULCA-Badge/VULCA-Badge.kicad_pcb (KiCad board)
At the start: 2 copper layers, 44.7 x 77.1 mm, 9 parts, among them SW1 SW_SPST

Commit message: Aligns all LEDs with the same orientation
Parts:
- Lg1: value LOGO -> F.Cu
- Lg2: value LOGO -> F.Mask
- Lg3: value LOGO -> B.Mask
- moved D1 2.15 mm to (126.7, 82.4), turned to 90 degrees
Connections:
- net Net-(BT1-+) renamed /3V2
- net Net-(D1-A) renamed /V+
Routing:
- net /V+: track 64.7 -> 71.5 mm
